File: Geiger/geiger/geiger.kicad_sch (KiCad schematic)
At the start: 21 parts, among them Q1 NMOS, U1 LM3478MA

Commit message: new files
Parts:
- added C10, C11, C12, C9: C, symbol Device:C
- added D9: D, symbol Device:D
- added L2: L, symbol Device:L
- added Q2: NMOS, symbol Simulation_SPICE:NMOS
- added R3, R4, R5, R6: R, symbol Device:R
Connections:
- net GND: now also C10.2, C11.2, C12.2, C9.2, R5.2, R6.2
- net VCC: now also U1.8 (V_{IN}), L2.1, Q2.1 (D)
- net at U1.1 (I_{SEN}): now also C9.1
- net at U1.2 (COMP): now also C11.1, R3.1
- net at U1.3 (FB): now also R4.2, R5.1
- net at U1.6 (DR): now also Q2.2 (G)
- new net: D9.2 (A), L2.2
- new net: Q2.3 (S), R6.1
- new net: C12.1, D9.1 (K), R4.1
- new net: C10.1, R3.2
Other:
- moved on the sheet: C1, C2, C3, C4, C5, C6, C7, C8, D1, D2, D3, D4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
