File: Stm32Board_Small_oneSide/Stm32Board.kicad_sch (KiCad schematic)
At the start: 57 parts, among them J1 USB_B_Micro, SW1 SW_Push, U1 STM32L151CBTx, U2 XC6210B332MR, Y1 32k, Y2 12Mhz

Commit message: new files
Parts:
- added U3: XC6206PxxxMR, Package_TO_SOT_SMD:SOT-23-3, symbol Regulator_Linear:XC6206PxxxMR
Connections:
- net +3.3V: now also U3.2 (VO)
- net GND: now also U3.1 (GND)
- net at C5.1, FB2.2, U2.1 (VIN)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: now also U3.3 (VI)
